File: main_controller/main_controller.kicad_sch (KiCad schematic)
At the start: 31 parts, among them J1 XH2.54 Male, J2 XH2.54 Male, J3 XH2.54 Male, SW1 SS12D01, SW10 Yellow, SW11 Green, SW2 SS12D01, SW3 SW_Push, SW4 SW_Push, SW6 Blue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

Commit message: finalize
Parts:
- added BT5: Lipo 1S 751640, symbol Device:Battery_Cell
- added SW12: SW_Push, symbol Switch:SW_Push
- added SW5: SS12D01, symbol Switch:SW_SPDT
Connections:
- net at SW2.3 (C): now also U2.19 (B+)
- net at U3.19 (B+): now also SW5.3 (C)
- net at U3.20 (B-): now also BT5.2 (-)
- net at U3.21 (RST): now also SW12.2
- net at U2.20 (B-): now also BT4.2 (-)
- new net: BT5.1 (+), SW5.2 (B)
Other:
- moved on the sheet: R4, R5, R6, R7, R8, R9, SW10, SW11, SW6, SW7, SW8, SW9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
